File: hardware/single_sh/single_sh.kicad_pcb (KiCad board)
At the start: 4 copper layers, 122 x 20 mm, 151 parts, among them J1 USB-C, J11 M1+M2, J12 M3+M4, J13 M5+M6, J14 M7+M8, J15 M9+M10, J2 Qwiic, J3 Qwiic, J4 5V IN, J5 LED STRIP, J6 LED PWR, J7 E-STOP, J8 PANEL BTN, Q1 AO3401A, SW1 BTN1, SW2 BTN2, SW3 BOOTSEL, U1 AT8833CQ, U10 AT8833CQ, U11 RP2354B, U12 TPD2E2U06, U13 ME6211C33M5G, U14 74AHCT1G125, U15 74AHCT1G125, U2 AT8833CQ, U3 AT8833CQ, U4 AT8833CQ, U5 AT8833CQ, U6 AT8833CQ, U7 AT8833CQ, U8 AT8833CQ, U9 AT8833CQ, Y1 12MHz

Commit message: single_sh: 0805 sense resistors; JLCPCB fab output
Sense resistors move from 0402 (62.5 mW) to 0805 (125 mW, Yageo
RL0805FR-070R82L, C513694); holding a coil at the current-limit trip is
now 56 % of rating. Driver-cell bottoms re-routed for the larger pads
(BOUT2 between the ISEN pads, BOUT1 under R_B), seven input nets
re-routed, motor labels moved onto the connectors. DRC: 0 unconnected,
no copper violations.

Also adds gen/jlcfab.py and the regenerated JLCPCB Gerbers/BOM/CPL.

Co-Authored-By: Claude Opus 5.5 <noreply@anthropic.com>
Parts:
- R1, R10, R11, R12, R13, R14, R15, R16, R17, R18, R19, R2, R20, R3, R4, R5, R6, R7, R8, R9: footprint Resistor_SMD:R_0402_1005Metric -> Resistor_SMD:R_0805_2012Metric
- moved R18 0.47 mm to (122.1, 103.3)
- moved R20 0.47 mm to (115.6, 103.3)
- moved R10 0.47 mm to (148.1, 103.3)
- moved R12 0.47 mm to (141.6, 103.3)
- moved R14 0.47 mm to (135.1, 103.3)
- moved R2 0.47 mm to (85.7, 103.3)
- moved R4 0.47 mm to (79.2, 103.3)
- moved R6 0.47 mm to (72.7, 103.3)
- moved R16 0.47 mm to (128.6, 103.3)
- moved R8 0.47 mm to (66.2, 103.3)
- moved R1 0.45 mm to (82.3, 103.3)
- moved R15 0.45 mm to (125.2, 103.3)
- moved R17 0.45 mm to (118.7, 103.3)
- moved R19 0.45 mm to (112.2, 103.3)
- moved R3 0.45 mm to (75.8, 103.3)
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Routing:
- net /M6_BIN2: track 43.6 -> 52.5 mm, vias 2 -> 6
- net /GND: track 113.7 -> 122.0 mm, vias 104 -> 102
- net /M3_BIN1: track 31.4 -> 37.7 mm
- net /M4_AIN2: track 43.3 -> 49.4 mm
- net /M6_AIN1: track 43.9 -> 45.7 mm
- net /M4_BIN1: track 50.9 -> 51.6 mm
- net /SWDIO: track 18.6 -> 19.1 mm

Commit message: single_sh: wired multi-sheet schematic
Replace the label-on-every-pin single_sh schematic with a presentable
hierarchical drawing: overview, power and USB, MCU, motor drivers,
connectors and UI (A3 sheets). Parts are wired, rails use power symbols,
inter-sheet signals use global labels, each block is framed with design
notes from the README.

- gen/schdraw.py draws wires/labels/power symbols and traces the drawing
  the way KiCad does; the build fails unless every pin is on the net
  build.py gave it. gen/single_sh_sch.py holds the layout.
- AT8833CQ gets a project symbol (lib/stack.kicad_sym, DRV8833RTY pin
  numbers) arranged so each driver cell draws without crossings.
- Same circuit: KiCad netlist has identical pin groupings, refs, values
  and footprints; BOM export unchanged; ERC 0.
- PCB re-linked to the new symbol paths and net names (/GND -> GND,
  locals -> /<sheet>/<name>); netclass patterns follow. Only path and net
  lines change. DRC unchanged (23 silk/courtyard warnings), 0 unconnected,
  0 parity issues. Fab outputs are exported without net names, so
  jlcpcb/ stays valid.

Co-Authored-By: Claude Opus 5.5 <noreply@anthropic.com>
Connections:
- net /+1V1 renamed +1V1
- net /+3V3 renamed +3V3
- net /+5V_EXT renamed /Power/+5V_EXT
- net /BOARD_ID renamed BOARD_ID
- net /BOOT_R renamed Net-(R36-Pad1)
- net /BTN1_N renamed Net-(R34-Pad1)
- net /BTN2_N renamed Net-(R35-Pad1)
- net /CC1 renamed CC1
- net /CC2 renamed CC2
- net /ESTOP_RET renamed Net-(J7-Pin_2)
- net /GND renamed GND
- net /I2C_PU renamed Net-(JP2-A)
- net /LADDER renamed LADDER
- net /LED_BUF renamed Net-(R38-Pad1)
- net /LED_DATA renamed /Connectors and UI/LED_DATA
- net /LED_DIN renamed LED_DIN
- net /LED_DIN_5V renamed Net-(D2-DIN)
- net /M10_AIN1 renamed M10_AIN1
- net /M10_AIN2 renamed M10_AIN2
- net /M10_AOUT1 renamed M10_AOUT1
- net /M10_AOUT2 renamed M10_AOUT2
- net /M10_BIN1 renamed M10_BIN1
- net /M10_BIN2 renamed M10_BIN2
- net /M10_BOUT1 renamed M10_BOUT1
- net /M10_BOUT2 renamed M10_BOUT2
- net /M1_AIN1 renamed M1_AIN1
- net /M1_AIN2 renamed M1_AIN2
- net /M1_AOUT1 renamed M1_AOUT1
- net /M1_AOUT2 renamed M1_AOUT2
- net /M1_BIN1 renamed M1_BIN1
- net /M1_BIN2 renamed M1_BIN2
- net /M1_BOUT1 renamed M1_BOUT1
- net /M1_BOUT2 renamed M1_BOUT2
- net /M2_AIN1 renamed M2_AIN1
- net /M2_AIN2 renamed M2_AIN2
- net /M2_AOUT1 renamed M2_AOUT1
- net /M2_AOUT2 renamed M2_AOUT2
- net /M2_BIN1 renamed M2_BIN1
- net /M2_BIN2 renamed M2_BIN2
- net /M2_BOUT1 renamed M2_BOUT1
- net /M2_BOUT2 renamed M2_BOUT2
- net /M3_AIN1 renamed M3_AIN1
- net /M3_AIN2 renamed M3_AIN2
- net /M3_AOUT1 renamed M3_AOUT1
- net /M3_AOUT2 renamed M3_AOUT2
- net /M3_BIN1 renamed M3_BIN1
- net /M3_BIN2 renamed M3_BIN2
- net /M3_BOUT1 renamed M3_BOUT1
- net /M3_BOUT2 renamed M3_BOUT2
- net /M4_AIN1 renamed M4_AIN1
- net /M4_AIN2 renamed M4_AIN2
- net /M4_AOUT1 renamed M4_AOUT1
- net /M4_AOUT2 renamed M4_AOUT2
- net /M4_BIN1 renamed M4_BIN1
- net /M4_BIN2 renamed M4_BIN2
- net /M4_BOUT1 renamed M4_BOUT1
- net /M4_BOUT2 renamed M4_BOUT2
- net /M5_AIN1 renamed M5_AIN1
- net /M5_AIN2 renamed M5_AIN2
- net /M5_AOUT1 renamed M5_AOUT1
- net /M5_AOUT2 renamed M5_AOUT2
- net /M5_BIN1 renamed M5_BIN1
- net /M5_BIN2 renamed M5_BIN2
- net /M5_BOUT1 renamed M5_BOUT1
- net /M5_BOUT2 renamed M5_BOUT2
- net /M6_AIN1 renamed M6_AIN1
- net /M6_AIN2 renamed M6_AIN2
- net /M6_AOUT1 renamed M6_AOUT1
- net /M6_AOUT2 renamed M6_AOUT2
- net /M6_BIN1 renamed M6_BIN1
- net /M6_BIN2 renamed M6_BIN2
- net /M6_BOUT1 renamed M6_BOUT1
- net /M6_BOUT2 renamed M6_BOUT2
- net /M7_AIN1 renamed M7_AIN1
- net /M7_AIN2 renamed M7_AIN2
- net /M7_AOUT1 renamed M7_AOUT1
- net /M7_AOUT2 renamed M7_AOUT2
- net /M7_BIN1 renamed M7_BIN1
- net /M7_BIN2 renamed M7_BIN2
- net /M7_BOUT1 renamed M7_BOUT1
- net /M7_BOUT2 renamed M7_BOUT2
- net /M8_AIN1 renamed M8_AIN1
- net /M8_AIN2 renamed M8_AIN2
- net /M8_AOUT1 renamed M8_AOUT1
- net /M8_AOUT2 renamed M8_AOUT2
- net /M8_BIN1 renamed M8_BIN1
- net /M8_BIN2 renamed M8_BIN2
- net /M8_BOUT1 renamed M8_BOUT1
- net /M8_BOUT2 renamed M8_BOUT2
- net /M9_AIN1 renamed M9_AIN1
- net /M9_AIN2 renamed M9_AIN2
- net /M9_AOUT1 renamed M9_AOUT1
- net /M9_AOUT2 renamed M9_AOUT2
- net /M9_BIN1 renamed M9_BIN1
- net /M9_BIN2 renamed M9_BIN2
- net /M9_BOUT1 renamed M9_BOUT1
- net /M9_BOUT2 renamed M9_BOUT2
- net /NSLEEP renamed /Motor drivers/NSLEEP
- net /PB1 renamed Net-(J8-Pin_2)
- net /PB2 renamed Net-(J8-Pin_3)
- net /QSPI_SS renamed /MCU/QSPI_SS
- net /QWIIC_3V3 renamed QWIIC_3V3
- net /RUN renamed /MCU/RUN
- net /SCL renamed SCL
- net /SDA renamed SDA
- net /SS_GATE renamed /Power/SS_GATE
- net /STRIP_5V renamed /Connectors and UI/STRIP_5V
- net /STRIP_DIN renamed /Connectors and UI/STRIP_DIN
- net /STRIP_V5_FUSED renamed /Connectors and UI/STRIP_V5_FUSED
- net /SWCLK renamed /MCU/SWCLK
- net /SWDIO renamed /MCU/SWDIO
- net /U10_AISEN renamed Net-(U10-AISEN)
- net /U10_BISEN renamed Net-(U10-BISEN)
- net /U10_VCP renamed Net-(U10-VCP)
- net /U10_VINT renamed Net-(U10-VINT)
- net /U1_AISEN renamed Net-(U1-AISEN)
- net /U1_BISEN renamed Net-(U1-BISEN)
- net /U1_VCP renamed Net-(U1-VCP)
- net /U1_VINT renamed Net-(U1-VINT)
- net /U2_AISEN renamed Net-(U2-AISEN)
- net /U2_BISEN renamed Net-(U2-BISEN)
- net /U2_VCP renamed Net-(U2-VCP)
- net /U2_VINT renamed Net-(U2-VINT)
- net /U3_AISEN renamed Net-(U3-AISEN)
- net /U3_BISEN renamed Net-(U3-BISEN)
- net /U3_VCP renamed Net-(U3-VCP)
- net /U3_VINT renamed Net-(U3-VINT)
- net /U4_AISEN renamed Net-(U4-AISEN)
- net /U4_BISEN renamed Net-(U4-BISEN)
- net /U4_VCP renamed Net-(U4-VCP)
- net /U4_VINT renamed Net-(U4-VINT)
- net /U5_AISEN renamed Net-(U5-AISEN)
- net /U5_BISEN renamed Net-(U5-BISEN)
- net /U5_VCP renamed Net-(U5-VCP)
- net /U5_VINT renamed Net-(U5-VINT)
- net /U6_AISEN renamed Net-(U6-AISEN)
- net /U6_BISEN renamed Net-(U6-BISEN)
- net /U6_VCP renamed Net-(U6-VCP)
- net /U6_VINT renamed Net-(U6-VINT)
- net /U7_AISEN renamed Net-(U7-AISEN)
- net /U7_BISEN renamed Net-(U7-BISEN)
- net /U7_VCP renamed Net-(U7-VCP)
- net /U7_VINT renamed Net-(U7-VINT)
- net /U8_AISEN renamed Net-(U8-AISEN)
- net /U8_BISEN renamed Net-(U8-BISEN)
- net /U8_VCP renamed Net-(U8-VCP)
- net /U8_VINT renamed Net-(U8-VINT)
- net /U9_AISEN renamed Net-(U9-AISEN)
- net /U9_BISEN renamed Net-(U9-BISEN)
- net /U9_VCP renamed Net-(U9-VCP)
- net /U9_VINT renamed Net-(U9-VINT)
- net /USB_DM renamed /Power/USB_DM
- net /USB_DM_MCU renamed USB_DM_MCU
- net /USB_DP renamed /Power/USB_DP
- net /USB_DP_MCU renamed USB_DP_MCU
- net /V5 renamed V5
- net /V5_IN renamed /Power/V5_IN
- net /VBUS renamed VBUS
- net /VBUS_F renamed /Power/VBUS_F
- net /VMOT_SENSE renamed VMOT_SENSE
- net /VREG_AVDD renamed /MCU/VREG_AVDD
- net /VREG_LX renamed /MCU/VREG_LX
- net /XIN renamed /MCU/XIN
- net /XOUT renamed /MCU/XOUT
- net /XTAL_OUT renamed /MCU/XTAL_OUT
