File: hardware/driver/driver.kicad_sch (KiCad schematic)
At the start: 71 parts, among them J1 BTB 40P socket, J2 BTB 40P socket, J3 BTB 40P header, J4 BTB 40P header, U1 AT8833CQ, U10 AT8833CQ, U2 AT8833CQ, U3 AT8833CQ, U4 AT8833CQ, U5 AT8833CQ, U6 AT8833CQ, U7 AT8833CQ, U8 AT8833CQ, U9 AT8833CQ

Commit message: single_sh: 0805 sense resistors; JLCPCB fab output
Sense resistors move from 0402 (62.5 mW) to 0805 (125 mW, Yageo
RL0805FR-070R82L, C513694); holding a coil at the current-limit trip is
now 56 % of rating. Driver-cell bottoms re-routed for the larger pads
(BOUT2 between the ISEN pads, BOUT1 under R_B), seven input nets
re-routed, motor labels moved onto the connectors. DRC: 0 unconnected,
no copper violations.

Also adds gen/jlcfab.py and the regenerated JLCPCB Gerbers/BOM/CPL.

Co-Authored-By: Claude Opus 5.5 <noreply@anthropic.com>
Parts:
- R1, R10, R11, R12, R13, R14, R15, R16, R17, R18, R19, R2, R20, R3, R4, R5, R6, R7, R8, R9: footprint Resistor_SMD:R_0402_1005Metric -> Resistor_SMD:R_0805_2012Metric; LCSC C728435 -> C513694; MPN RL0402FR-070R82L -> RL0805FR-070R82L
Changed lines of the file:
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@@
 			)
 		)
-		(property "Footprint" "Resistor_SMD:R_0402_1005Metric"
+		(property "Footprint" "Resistor_SMD:R_0805_2012Metric"
 			(at 116.84 40.64 0)
 			(hide yes)
@@
 			)
 		)
-		(property "LCSC" "C728435"
+		(property "LCSC" "C513694"
 			(at 116.84 40.64 0)
 			(hide yes)
@@
 			)
 		)
-		(property "MPN" "RL0402FR-070R82L"
+		(property "MPN" "RL0805FR-070R82L"
 			(at 116.84 40.64 0)
 			(hide yes)
@@
 			)
 		)
-		(property "Footprint" "Resistor_SMD:R_0402_1005Metric"
+		(property "Footprint" "Resistor_SMD:R_0805_2012Metric"
 			(at 167.64 40.64 0)
 			(hide yes)
@@
 			)
 		)
-		(property "LCSC" "C728435"
+		(property "LCSC" "C513694"
 			(at 167.64 40.64 0)
 			(hide yes)
@@
 			)
 		)
-		(property "MPN" "RL0402FR-070R82L"
+		(property "MPN" "RL0805FR-070R82L"
 			(at 167.64 40.64 0)
 			(hide yes)
@@
 			)
 		)
-		(property "Footprint" "Resistor_SMD:R_0402_1005Metric"
+		(property "Footprint" "Resistor_SMD:R_0805_2012Metric"
 			(at 492.76 40.64 0)
 			(hide yes)
@@
 			)
 		)
-		(property "LCSC" "C728435"
+		(property "LCSC" "C513694"
 			(at 492.76 40.64 0)
 			(hide yes)
@@
 			)
 		)
-		(property "MPN" "RL0402FR-070R82L"
+		(property "MPN" "RL0805FR-070R82L"
 			(at 492.76 40.64 0)
 			(hide yes)
@@
 			)
 		)
-		(property "Footprint" "Resistor_SMD:R_0402_1005Metric"
+		(property "Footprint" "Resistor_SMD:R_0805_2012Metric"
 			(at 43.18 86.36 0)
 			(hide yes)
@@
 			)
 		)
-		(property "LCSC" "C728435"
+		(property "LCSC" "C513694"
 			(at 43.18 86.36 0)
 			(hide yes)
@@
 			)
 		)
-		(property "MPN" "RL0402FR-070R82L"
+		(property "MPN" "RL0805FR-070R82L"
 			(at 43.18 86.36 0)
 			(hide yes)
@@
 			)
 		)
-		(property "Footprint" "Resistor_SMD:R_0402_1005Metric"
+		(property "Footprint" "Resistor_SMD:R_0805_2012Metric"
 			(at 368.3 86.36 0)
 			(hide yes)
@@
 			)
 		)
-		(property "LCSC" "C728435"
+		(property "LCSC" "C513694"
 			(at 368.3 86.36 0)
 			(hide yes)
@@
 			)
 		)
-		(property "MPN" "RL0402FR-070R82L"
+		(property "MPN" "RL0805FR-070R82L"
 			(at 368.3 86.36 0)
 			(hide yes)
@@
 			)
 		)
-		(property "Footprint" "Resistor_SMD:R_0402_1005Metric"
+		(property "Footprint" "Resistor_SMD:R_0805_2012Metric"
 			(at 416.56 86.36 0)
 			(hide yes)
@@
 			)
 		)
-		(property "LCSC" "C728435"
+		(property "LCSC" "C513694"
 			(at 416.56 86.36 0)
 			(hide yes)
@@
 			)
 		)
-		(property "MPN" "RL0402FR-070R82L"
+		(property "MPN" "RL0805FR-070R82L"
 			(at 416.56 86.36 0)
 			(hide yes)
@@
 			)
 		)
-		(property "Footprint" "Resistor_SMD:R_0402_1005Metric"
+		(property "Footprint" "Resistor_SMD:R_0805_2012Metric"
 			(at 218.44 129.54 0)
 			(hide yes)
@@
 			)
 		)
-		(property "LCSC" "C728435"
+		(property "LCSC" "C513694"
 			(at 218.44 129.54 0)
 			(hide yes)
@@
 			)
 		)
-		(property "MPN" "RL0402FR-070R82L"
+		(property "MPN" "RL0805FR-070R82L"
 			(at 218.44 129.54 0)
 			(hide yes)
@@
 			)
 		)
-		(property "Footprint" "Resistor_SMD:R_0402_1005Metric"
+		(property "Footprint" "Resistor_SMD:R_0805_2012Metric"
 			(at 266.7 129.54 0)
 			(hide yes)
@@
 			)
 		)
-		(property "LCSC" "C728435"
+		(property "LCSC" "C513694"
 			(at 266.7 129.54 0)
 			(hide yes)
@@
 			)
 		)
-		(property "MPN" "RL0402FR-070R82L"
+		(property "MPN" "RL0805FR-070R82L"
 			(at 266.7 129.54 0)
 			(hide yes)
@@
 			)
 		)
-		(property "Footprint" "Resistor_SMD:R_0402_1005Metric"
+		(property "Footprint" "Resistor_SMD:R_0805_2012Metric"
 			(at 116.84 175.26 0)
 			(hide yes)
@@
 			)
 		)
-		(property "LCSC" "C728435"
+		(property "LCSC" "C513694"
 			(at 116.84 175.26 0)
 			(hide yes)
@@
 			)
 		)
-		(property "MPN" "RL0402FR-070R82L"
+		(property "MPN" "RL0805FR-070R82L"
 			(at 116.84 175.26 0)
 			(hide yes)
@@
 			)
 		)
-		(property "Footprint" "Resistor_SMD:R_0402_1005Metric"
+		(property "Footprint" "Resistor_SMD:R_0805_2012Metric"
 			(at 167.64 175.26 0)
 			(hide yes)
@@
 			)
 		)
-		(property "LCSC" "C728435"
+		(property "LCSC" "C513694"
 			(at 167.64 175.26 0)
 			(hide yes)
@@
 			)
 		)
-		(property "MPN" "RL0402FR-070R82L"
+		(property "MPN" "RL0805FR-070R82L"
 			(at 167.64 175.26 0)
 			(hide yes)
@@
 			)
 		)
-		(property "Footprint" "Resistor_SMD:R_0402_1005Metric"
+		(property "Footprint" "Resistor_SMD:R_0805_2012Metric"
 			(at 492.76 175.26 0)
 			(hide yes)
@@
 			)
 		)
-		(property "LCSC" "C728435"
+		(property "LCSC" "C513694"
 			(at 492.76 175.26 0)
 			(hide yes)
@@
 			)
 		)
-		(property "MPN" "RL0402FR-070R82L"
+		(property "MPN" "RL0805FR-070R82L"
 			(at 492.76 175.26 0)
 			(hide yes)
@@
 			)
 		)
-		(property "Footprint" "Resistor_SMD:R_0402_1005Metric"
+		(property "Footprint" "Resistor_SMD:R_0805_2012Metric"
 			(at 43.18 220.98 0)
 			(hide yes)
@@
 			)
 		)
-		(property "LCSC" "C728435"
+		(property "LCSC" "C513694"
 			(at 43.18 220.98 0)
 			(hide yes)
@@
 			)
 		)
-		(property "MPN" "RL0402FR-070R82L"
+		(property "MPN" "RL0805FR-070R82L"
 			(at 43.18 220.98 0)
 			(hide yes)
@@
 			)
 		)
-		(property "Footprint" "Resistor_SMD:R_0402_1005Metric"
+		(property "Footprint" "Resistor_SMD:R_0805_2012Metric"
 			(at 368.3 220.98 0)
 			(hide yes)
@@
 			)
 		)
-		(property "LCSC" "C728435"
+		(property "LCSC" "C513694"
 			(at 368.3 220.98 0)
 			(hide yes)
@@
 			)
 		)
-		(property "MPN" "RL0402FR-070R82L"
+		(property "MPN" "RL0805FR-070R82L"
 			(at 368.3 220.98 0)
 			(hide yes)
@@
 			)
 		)
-		(property "Footprint" "Resistor_SMD:R_0402_1005Metric"
+		(property "Footprint" "Resistor_SMD:R_0805_2012Metric"
 			(at 416.56 220.98 0)
 			(hide yes)
@@
 			)
 		)
-		(property "LCSC" "C728435"
+		(property "LCSC" "C513694"
 			(at 416.56 220.98 0)
 			(hide yes)
@@
 			)
 		)
-		(property "MPN" "RL0402FR-070R82L"
+		(property "MPN" "RL0805FR-070R82L"
 			(at 416.56 220.98 0)
 			(hide yes)
@@
 			)
 		)
-		(property "Footprint" "Resistor_SMD:R_0402_1005Metric"
+		(property "Footprint" "Resistor_SMD:R_0805_2012Metric"
 			(at 218.44 264.16 0)
 			(hide yes)
@@
 			)
 		)
-		(property "LCSC" "C728435"
+		(property "LCSC" "C513694"
 			(at 218.44 264.16 0)
 			(hide yes)
@@
 			)
 		)
-		(property "MPN" "RL0402FR-070R82L"
+		(property "MPN" "RL0805FR-070R82L"
 			(at 218.44 264.16 0)
 			(hide yes)
@@
 			)
 		)
-		(property "Footprint" "Resistor_SMD:R_0402_1005Metric"
+		(property "Footprint" "Resistor_SMD:R_0805_2012Metric"
 			(at 266.7 264.16 0)
 			(hide yes)
@@
 			)
 		)
-		(property "LCSC" "C728435"
+		(property "LCSC" "C513694"
 			(at 266.7 264.16 0)
 			(hide yes)
@@
 			)
 		)
-		(property "MPN" "RL0402FR-070R82L"
+		(property "MPN" "RL0805FR-070R82L"
 			(at 266.7 264.16 0)
 			(hide yes)
@@
 			)
 		)
-		(property "Footprint" "Resistor_SMD:R_0402_1005Metric"
+		(property "Footprint" "Resistor_SMD:R_0805_2012Metric"
 			(at 116.84 309.88 0)
 			(hide yes)
@@
 			)
 		)
-		(property "LCSC" "C728435"
+		(property "LCSC" "C513694"
 			(at 116.84 309.88 0)
 			(hide yes)
@@
 			)
 		)
-		(property "MPN" "RL0402FR-070R82L"
+		(property "MPN" "RL0805FR-070R82L"
 			(at 116.84 309.88 0)
 			(hide yes)
@@
 			)
 		)
-		(property "Footprint" "Resistor_SMD:R_0402_1005Metric"
+		(property "Footprint" "Resistor_SMD:R_0805_2012Metric"
 			(at 167.64 309.88 0)
 			(hide yes)
@@
 			)
 		)
-		(property "LCSC" "C728435"
+		(property "LCSC" "C513694"
 			(at 167.64 309.88 0)
 			(hide yes)
@@
 			)
 		)
-		(property "MPN" "RL0402FR-070R82L"
+		(property "MPN" "RL0805FR-070R82L"
 			(at 167.64 309.88 0)
 			(hide yes)
@@
 			)
 		)
-		(property "Footprint" "Resistor_SMD:R_0402_1005Metric"
+		(property "Footprint" "Resistor_SMD:R_0805_2012Metric"
 			(at 492.76 309.88 0)
 			(hide yes)
@@
 			)
 		)
-		(property "LCSC" "C728435"
+		(property "LCSC" "C513694"
 			(at 492.76 309.88 0)
 			(hide yes)
@@
 			)
 		)
-		(property "MPN" "RL0402FR-070R82L"
+		(property "MPN" "RL0805FR-070R82L"
 			(at 492.76 309.88 0)
 			(hide yes)
@@
 			)
 		)
-		(property "Footprint" "Resistor_SMD:R_0402_1005Metric"
+		(property "Footprint" "Resistor_SMD:R_0805_2012Metric"
 			(at 43.18 353.06 0)
 			(hide yes)
@@
 			)
 		)
-		(property "LCSC" "C728435"
+		(property "LCSC" "C513694"
 			(at 43.18 353.06 0)
 			(hide yes)
@@
 			)
 		)
-		(property "MPN" "RL0402FR-070R82L"
+		(property "MPN" "RL0805FR-070R82L"
 			(at 43.18 353.06 0)
 			(hide yes)

Commit message: single_sh: 0603 sense resistors; refilled zones, fab output
Sense resistors move from 0805 to 0603 (Viking SR731JTTDR820F, C186570,
250 mW); holding a coil at the current-limit trip is now 28 % of rating.
Swapped in place on the routed board: ISEN pad kept, GND pad 0.275 mm
inboard (R5/R11 keep the GND pad instead). Zones refilled after the route
cleanup and trace edits. DRC: 0 unconnected, 0 parity, no copper
violations; 4 silkscreen warnings.

Schematics, BOMs, generators and README updated; JLCPCB Gerbers/BOM/CPL
regenerated and placement-checked.

Co-Authored-By: Claude Opus 5.5 <noreply@anthropic.com>
Parts:
- R1, R10, R11, R12, R13, R14, R15, R16, R17, R18, R19, R2, R20, R3, R4, R5, R6, R7, R8, R9: footprint Resistor_SMD:R_0805_2012Metric -> Resistor_SMD:R_0603_1608Metric; LCSC C513694 -> C186570; MPN RL0805FR-070R82L -> SR731JTTDR820F
Changed lines of the file:
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@@
 			)
 		)
-		(property "Footprint" "Resistor_SMD:R_0805_2012Metric"
+		(property "Footprint" "Resistor_SMD:R_0603_1608Metric"
 			(at 116.84 40.64 0)
 			(hide yes)
@@
 			)
 		)
-		(property "LCSC" "C513694"
+		(property "LCSC" "C186570"
 			(at 116.84 40.64 0)
 			(hide yes)
@@
 			)
 		)
-		(property "MPN" "RL0805FR-070R82L"
+		(property "MPN" "SR731JTTDR820F"
 			(at 116.84 40.64 0)
 			(hide yes)
@@
 			)
 		)
-		(property "Footprint" "Resistor_SMD:R_0805_2012Metric"
+		(property "Footprint" "Resistor_SMD:R_0603_1608Metric"
 			(at 167.64 40.64 0)
 			(hide yes)
@@
 			)
 		)
-		(property "LCSC" "C513694"
+		(property "LCSC" "C186570"
 			(at 167.64 40.64 0)
 			(hide yes)
@@
 			)
 		)
-		(property "MPN" "RL0805FR-070R82L"
+		(property "MPN" "SR731JTTDR820F"
 			(at 167.64 40.64 0)
 			(hide yes)
@@
 			)
 		)
-		(property "Footprint" "Resistor_SMD:R_0805_2012Metric"
+		(property "Footprint" "Resistor_SMD:R_0603_1608Metric"
 			(at 492.76 40.64 0)
 			(hide yes)
@@
 			)
 		)
-		(property "LCSC" "C513694"
+		(property "LCSC" "C186570"
 			(at 492.76 40.64 0)
 			(hide yes)
@@
 			)
 		)
-		(property "MPN" "RL0805FR-070R82L"
+		(property "MPN" "SR731JTTDR820F"
 			(at 492.76 40.64 0)
 			(hide yes)
@@
 			)
 		)
-		(property "Footprint" "Resistor_SMD:R_0805_2012Metric"
+		(property "Footprint" "Resistor_SMD:R_0603_1608Metric"
 			(at 43.18 86.36 0)
 			(hide yes)
@@
 			)
 		)
-		(property "LCSC" "C513694"
+		(property "LCSC" "C186570"
 			(at 43.18 86.36 0)
 			(hide yes)
@@
 			)
 		)
-		(property "MPN" "RL0805FR-070R82L"
+		(property "MPN" "SR731JTTDR820F"
 			(at 43.18 86.36 0)
 			(hide yes)
@@
 			)
 		)
-		(property "Footprint" "Resistor_SMD:R_0805_2012Metric"
+		(property "Footprint" "Resistor_SMD:R_0603_1608Metric"
 			(at 368.3 86.36 0)
 			(hide yes)
@@
 			)
 		)
-		(property "LCSC" "C513694"
+		(property "LCSC" "C186570"
 			(at 368.3 86.36 0)
 			(hide yes)
@@
 			)
 		)
-		(property "MPN" "RL0805FR-070R82L"
+		(property "MPN" "SR731JTTDR820F"
 			(at 368.3 86.36 0)
 			(hide yes)
@@
 			)
 		)
-		(property "Footprint" "Resistor_SMD:R_0805_2012Metric"
+		(property "Footprint" "Resistor_SMD:R_0603_1608Metric"
 			(at 416.56 86.36 0)
 			(hide yes)
@@
 			)
 		)
-		(property "LCSC" "C513694"
+		(property "LCSC" "C186570"
 			(at 416.56 86.36 0)
 			(hide yes)
@@
 			)
 		)
-		(property "MPN" "RL0805FR-070R82L"
+		(property "MPN" "SR731JTTDR820F"
 			(at 416.56 86.36 0)
 			(hide yes)
@@
 			)
 		)
-		(property "Footprint" "Resistor_SMD:R_0805_2012Metric"
+		(property "Footprint" "Resistor_SMD:R_0603_1608Metric"
 			(at 218.44 129.54 0)
 			(hide yes)
@@
 			)
 		)
-		(property "LCSC" "C513694"
+		(property "LCSC" "C186570"
 			(at 218.44 129.54 0)
 			(hide yes)
@@
 			)
 		)
-		(property "MPN" "RL0805FR-070R82L"
+		(property "MPN" "SR731JTTDR820F"
 			(at 218.44 129.54 0)
 			(hide yes)
@@
 			)
 		)
-		(property "Footprint" "Resistor_SMD:R_0805_2012Metric"
+		(property "Footprint" "Resistor_SMD:R_0603_1608Metric"
 			(at 266.7 129.54 0)
 			(hide yes)
@@
 			)
 		)
-		(property "LCSC" "C513694"
+		(property "LCSC" "C186570"
 			(at 266.7 129.54 0)
 			(hide yes)
@@
 			)
 		)
-		(property "MPN" "RL0805FR-070R82L"
+		(property "MPN" "SR731JTTDR820F"
 			(at 266.7 129.54 0)
 			(hide yes)
@@
 			)
 		)
-		(property "Footprint" "Resistor_SMD:R_0805_2012Metric"
+		(property "Footprint" "Resistor_SMD:R_0603_1608Metric"
 			(at 116.84 175.26 0)
 			(hide yes)
@@
 			)
 		)
-		(property "LCSC" "C513694"
+		(property "LCSC" "C186570"
 			(at 116.84 175.26 0)
 			(hide yes)
@@
 			)
 		)
-		(property "MPN" "RL0805FR-070R82L"
+		(property "MPN" "SR731JTTDR820F"
 			(at 116.84 175.26 0)
 			(hide yes)
@@
 			)
 		)
-		(property "Footprint" "Resistor_SMD:R_0805_2012Metric"
+		(property "Footprint" "Resistor_SMD:R_0603_1608Metric"
 			(at 167.64 175.26 0)
 			(hide yes)
@@
 			)
 		)
-		(property "LCSC" "C513694"
+		(property "LCSC" "C186570"
 			(at 167.64 175.26 0)
 			(hide yes)
@@
 			)
 		)
-		(property "MPN" "RL0805FR-070R82L"
+		(property "MPN" "SR731JTTDR820F"
 			(at 167.64 175.26 0)
 			(hide yes)
@@
 			)
 		)
-		(property "Footprint" "Resistor_SMD:R_0805_2012Metric"
+		(property "Footprint" "Resistor_SMD:R_0603_1608Metric"
 			(at 492.76 175.26 0)
 			(hide yes)
@@
 			)
 		)
-		(property "LCSC" "C513694"
+		(property "LCSC" "C186570"
 			(at 492.76 175.26 0)
 			(hide yes)
@@
 			)
 		)
-		(property "MPN" "RL0805FR-070R82L"
+		(property "MPN" "SR731JTTDR820F"
 			(at 492.76 175.26 0)
 			(hide yes)
@@
 			)
 		)
-		(property "Footprint" "Resistor_SMD:R_0805_2012Metric"
+		(property "Footprint" "Resistor_SMD:R_0603_1608Metric"
 			(at 43.18 220.98 0)
 			(hide yes)
@@
 			)
 		)
-		(property "LCSC" "C513694"
+		(property "LCSC" "C186570"
 			(at 43.18 220.98 0)
 			(hide yes)
@@
 			)
 		)
-		(property "MPN" "RL0805FR-070R82L"
+		(property "MPN" "SR731JTTDR820F"
 			(at 43.18 220.98 0)
 			(hide yes)
@@
 			)
 		)
-		(property "Footprint" "Resistor_SMD:R_0805_2012Metric"
+		(property "Footprint" "Resistor_SMD:R_0603_1608Metric"
 			(at 368.3 220.98 0)
 			(hide yes)
@@
 			)
 		)
-		(property "LCSC" "C513694"
+		(property "LCSC" "C186570"
 			(at 368.3 220.98 0)
 			(hide yes)
@@
 			)
 		)
-		(property "MPN" "RL0805FR-070R82L"
+		(property "MPN" "SR731JTTDR820F"
 			(at 368.3 220.98 0)
 			(hide yes)
@@
 			)
 		)
-		(property "Footprint" "Resistor_SMD:R_0805_2012Metric"
+		(property "Footprint" "Resistor_SMD:R_0603_1608Metric"
 			(at 416.56 220.98 0)
 			(hide yes)
@@
 			)
 		)
-		(property "LCSC" "C513694"
+		(property "LCSC" "C186570"
 			(at 416.56 220.98 0)
 			(hide yes)
@@
 			)
 		)
-		(property "MPN" "RL0805FR-070R82L"
+		(property "MPN" "SR731JTTDR820F"
 			(at 416.56 220.98 0)
 			(hide yes)
@@
 			)
 		)
-		(property "Footprint" "Resistor_SMD:R_0805_2012Metric"
+		(property "Footprint" "Resistor_SMD:R_0603_1608Metric"
 			(at 218.44 264.16 0)
 			(hide yes)
@@
 			)
 		)
-		(property "LCSC" "C513694"
+		(property "LCSC" "C186570"
 			(at 218.44 264.16 0)
 			(hide yes)
@@
 			)
 		)
-		(property "MPN" "RL0805FR-070R82L"
+		(property "MPN" "SR731JTTDR820F"
 			(at 218.44 264.16 0)
 			(hide yes)
@@
 			)
 		)
-		(property "Footprint" "Resistor_SMD:R_0805_2012Metric"
+		(property "Footprint" "Resistor_SMD:R_0603_1608Metric"
 			(at 266.7 264.16 0)
 			(hide yes)
@@
 			)
 		)
-		(property "LCSC" "C513694"
+		(property "LCSC" "C186570"
 			(at 266.7 264.16 0)
 			(hide yes)
@@
 			)
 		)
-		(property "MPN" "RL0805FR-070R82L"
+		(property "MPN" "SR731JTTDR820F"
 			(at 266.7 264.16 0)
 			(hide yes)
@@
 			)
 		)
-		(property "Footprint" "Resistor_SMD:R_0805_2012Metric"
+		(property "Footprint" "Resistor_SMD:R_0603_1608Metric"
 			(at 116.84 309.88 0)
 			(hide yes)
@@
 			)
 		)
-		(property "LCSC" "C513694"
+		(property "LCSC" "C186570"
 			(at 116.84 309.88 0)
 			(hide yes)
@@
 			)
 		)
-		(property "MPN" "RL0805FR-070R82L"
+		(property "MPN" "SR731JTTDR820F"
 			(at 116.84 309.88 0)
 			(hide yes)
@@
 			)
 		)
-		(property "Footprint" "Resistor_SMD:R_0805_2012Metric"
+		(property "Footprint" "Resistor_SMD:R_0603_1608Metric"
 			(at 167.64 309.88 0)
 			(hide yes)
@@
 			)
 		)
-		(property "LCSC" "C513694"
+		(property "LCSC" "C186570"
 			(at 167.64 309.88 0)
 			(hide yes)
@@
 			)
 		)
-		(property "MPN" "RL0805FR-070R82L"
+		(property "MPN" "SR731JTTDR820F"
 			(at 167.64 309.88 0)
 			(hide yes)
@@
 			)
 		)
-		(property "Footprint" "Resistor_SMD:R_0805_2012Metric"
+		(property "Footprint" "Resistor_SMD:R_0603_1608Metric"
 			(at 492.76 309.88 0)
 			(hide yes)
@@
 			)
 		)
-		(property "LCSC" "C513694"
+		(property "LCSC" "C186570"
 			(at 492.76 309.88 0)
 			(hide yes)
@@
 			)
 		)
-		(property "MPN" "RL0805FR-070R82L"
+		(property "MPN" "SR731JTTDR820F"
 			(at 492.76 309.88 0)
 			(hide yes)
@@
 			)
 		)
-		(property "Footprint" "Resistor_SMD:R_0805_2012Metric"
+		(property "Footprint" "Resistor_SMD:R_0603_1608Metric"
 			(at 43.18 353.06 0)
 			(hide yes)
@@
 			)
 		)
-		(property "LCSC" "C513694"
+		(property "LCSC" "C186570"
 			(at 43.18 353.06 0)
 			(hide yes)
@@
 			)
 		)
-		(property "MPN" "RL0805FR-070R82L"
+		(property "MPN" "SR731JTTDR820F"
 			(at 43.18 353.06 0)
 			(hide yes)

Commit message: single_sh_proto: all-0603 basic-parts prototype board, as ordered
150 x 30 mm 4-layer board, fully routed (0.52/0.3 vias, 45-degree traces,
centred pad entries, no vias in pads), JLCDFM clean. Corrected nested
dual-motor connector pinout, bring-up test points, back-silk squid art.
L1 substituted (C411344); status LED D2 is the 5050 WS2812B (C2843785),
left off the Economic PCBA order for hand soldering.

Generator updates for the proto board (build.py, pcbgen.py, jlcfab.py,
single_sh_sch.py, add_testpoints.py, squid_silk.py) and regenerated
outputs for the other boards.

Ordered from JLCPCB 2026-10-11: 5 boards, Economic PCBA.

Co-Authored-By: Claude Opus 5.5 <noreply@anthropic.com>
Parts:
- R1, R10, R11, R12, R13, R14, R15, R16, R17, R18, R19, R2, R20, R3, R4, R5, R6, R7, R8, R9: value 0.82 -> 1; LCSC C186570 -> C22936; MPN SR731JTTDR820F -> 0603WAF100KT5E; Note chops at 0.2-0.29 A (VTRIP 160-240 mV); Kelvin return -> chops at 0.16-0.24 A (VTRIP 160-240 mV); Kelvin return
