File: hardware/single_xh/single_xh.kicad_sch (KiCad schematic)
At the start: 156 parts, among them J1 USB-C, J11 M1, J12 M2, J13 M3, J14 M4, J15 M5, J16 M6, J17 M7, J18 M8, J19 M9, J2 Qwiic, J20 M10, J3 Qwiic, J4 5V IN, J5 LED STRIP, J6 LED PWR, J7 E-STOP, J8 PANEL BTN, Q1 AO3401A, SW1 BTN1, SW2 BTN2, SW3 BOOTSEL, U1 AT8833CQ, U10 AT8833CQ, U11 RP2354B, U12 TPD2E2U06, U13 ME6211C33M5G, U14 74AHCT1G125, U15 74AHCT1G125, U2 AT8833CQ, U3 AT8833CQ, U4 AT8833CQ, U5 AT8833CQ, U6 AT8833CQ, U7 AT8833CQ, U8 AT8833CQ, U9 AT8833CQ, Y1 12MHz

Commit message: single_sh: 0805 sense resistors; JLCPCB fab output
Sense resistors move from 0402 (62.5 mW) to 0805 (125 mW, Yageo
RL0805FR-070R82L, C513694); holding a coil at the current-limit trip is
now 56 % of rating. Driver-cell bottoms re-routed for the larger pads
(BOUT2 between the ISEN pads, BOUT1 under R_B), seven input nets
re-routed, motor labels moved onto the connectors. DRC: 0 unconnected,
no copper violations.

Also adds gen/jlcfab.py and the regenerated JLCPCB Gerbers/BOM/CPL.

Co-Authored-By: Claude Opus 5.5 <noreply@anthropic.com>
Parts:
- R1, R10, R11, R12, R13, R14, R15, R16, R17, R18, R19, R2, R20, R3, R4, R5, R6, R7, R8, R9: footprint Resistor_SMD:R_0402_1005Metric -> Resistor_SMD:R_0805_2012Metric; LCSC C728435 -> C513694; MPN RL0402FR-070R82L -> RL0805FR-070R82L
Changed lines of the file:
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@@
 			)
 		)
-		(property "Footprint" "Resistor_SMD:R_0402_1005Metric"
+		(property "Footprint" "Resistor_SMD:R_0805_2012Metric"
 			(at 116.84 40.64 0)
 			(hide yes)
@@
 			)
 		)
-		(property "LCSC" "C728435"
+		(property "LCSC" "C513694"
 			(at 116.84 40.64 0)
 			(hide yes)
@@
 			)
 		)
-		(property "MPN" "RL0402FR-070R82L"
+		(property "MPN" "RL0805FR-070R82L"
 			(at 116.84 40.64 0)
 			(hide yes)
@@
 			)
 		)
-		(property "Footprint" "Resistor_SMD:R_0402_1005Metric"
+		(property "Footprint" "Resistor_SMD:R_0805_2012Metric"
 			(at 167.64 40.64 0)
 			(hide yes)
@@
 			)
 		)
-		(property "LCSC" "C728435"
+		(property "LCSC" "C513694"
 			(at 167.64 40.64 0)
 			(hide yes)
@@
 			)
 		)
-		(property "MPN" "RL0402FR-070R82L"
+		(property "MPN" "RL0805FR-070R82L"
 			(at 167.64 40.64 0)
 			(hide yes)
@@
 			)
 		)
-		(property "Footprint" "Resistor_SMD:R_0402_1005Metric"
+		(property "Footprint" "Resistor_SMD:R_0805_2012Metric"
 			(at 492.76 40.64 0)
 			(hide yes)
@@
 			)
 		)
-		(property "LCSC" "C728435"
+		(property "LCSC" "C513694"
 			(at 492.76 40.64 0)
 			(hide yes)
@@
 			)
 		)
-		(property "MPN" "RL0402FR-070R82L"
+		(property "MPN" "RL0805FR-070R82L"
 			(at 492.76 40.64 0)
 			(hide yes)
@@
 			)
 		)
-		(property "Footprint" "Resistor_SMD:R_0402_1005Metric"
+		(property "Footprint" "Resistor_SMD:R_0805_2012Metric"
 			(at 543.56 40.64 0)
 			(hide yes)
@@
 			)
 		)
-		(property "LCSC" "C728435"
+		(property "LCSC" "C513694"
 			(at 543.56 40.64 0)
 			(hide yes)
@@
 			)
 		)
-		(property "MPN" "RL0402FR-070R82L"
+		(property "MPN" "RL0805FR-070R82L"
 			(at 543.56 40.64 0)
 			(hide yes)
@@
 			)
 		)
-		(property "Footprint" "Resistor_SMD:R_0402_1005Metric"
+		(property "Footprint" "Resistor_SMD:R_0805_2012Metric"
 			(at 116.84 86.36 0)
 			(hide yes)
@@
 			)
 		)
-		(property "LCSC" "C728435"
+		(property "LCSC" "C513694"
 			(at 116.84 86.36 0)
 			(hide yes)
@@
 			)
 		)
-		(property "MPN" "RL0402FR-070R82L"
+		(property "MPN" "RL0805FR-070R82L"
 			(at 116.84 86.36 0)
 			(hide yes)
@@
 			)
 		)
-		(property "Footprint" "Resistor_SMD:R_0402_1005Metric"
+		(property "Footprint" "Resistor_SMD:R_0805_2012Metric"
 			(at 167.64 86.36 0)
 			(hide yes)
@@
 			)
 		)
-		(property "LCSC" "C728435"
+		(property "LCSC" "C513694"
 			(at 167.64 86.36 0)
 			(hide yes)
@@
 			)
 		)
-		(property "MPN" "RL0402FR-070R82L"
+		(property "MPN" "RL0805FR-070R82L"
 			(at 167.64 86.36 0)
 			(hide yes)
@@
 			)
 		)
-		(property "Footprint" "Resistor_SMD:R_0402_1005Metric"
+		(property "Footprint" "Resistor_SMD:R_0805_2012Metric"
 			(at 492.76 86.36 0)
 			(hide yes)
@@
 			)
 		)
-		(property "LCSC" "C728435"
+		(property "LCSC" "C513694"
 			(at 492.76 86.36 0)
 			(hide yes)
@@
 			)
 		)
-		(property "MPN" "RL0402FR-070R82L"
+		(property "MPN" "RL0805FR-070R82L"
 			(at 492.76 86.36 0)
 			(hide yes)
@@
 			)
 		)
-		(property "Footprint" "Resistor_SMD:R_0402_1005Metric"
+		(property "Footprint" "Resistor_SMD:R_0805_2012Metric"
 			(at 543.56 86.36 0)
 			(hide yes)
@@
 			)
 		)
-		(property "LCSC" "C728435"
+		(property "LCSC" "C513694"
 			(at 543.56 86.36 0)
 			(hide yes)
@@
 			)
 		)
-		(property "MPN" "RL0402FR-070R82L"
+		(property "MPN" "RL0805FR-070R82L"
 			(at 543.56 86.36 0)
 			(hide yes)
@@
 			)
 		)
-		(property "Footprint" "Resistor_SMD:R_0402_1005Metric"
+		(property "Footprint" "Resistor_SMD:R_0805_2012Metric"
 			(at 116.84 129.54 0)
 			(hide yes)
@@
 			)
 		)
-		(property "LCSC" "C728435"
+		(property "LCSC" "C513694"
 			(at 116.84 129.54 0)
 			(hide yes)
@@
 			)
 		)
-		(property "MPN" "RL0402FR-070R82L"
+		(property "MPN" "RL0805FR-070R82L"
 			(at 116.84 129.54 0)
 			(hide yes)
@@
 			)
 		)
-		(property "Footprint" "Resistor_SMD:R_0402_1005Metric"
+		(property "Footprint" "Resistor_SMD:R_0805_2012Metric"
 			(at 167.64 129.54 0)
 			(hide yes)
@@
 			)
 		)
-		(property "LCSC" "C728435"
+		(property "LCSC" "C513694"
 			(at 167.64 129.54 0)
 			(hide yes)
@@
 			)
 		)
-		(property "MPN" "RL0402FR-070R82L"
+		(property "MPN" "RL0805FR-070R82L"
 			(at 167.64 129.54 0)
 			(hide yes)
@@
 			)
 		)
-		(property "Footprint" "Resistor_SMD:R_0402_1005Metric"
+		(property "Footprint" "Resistor_SMD:R_0805_2012Metric"
 			(at 492.76 129.54 0)
 			(hide yes)
@@
 			)
 		)
-		(property "LCSC" "C728435"
+		(property "LCSC" "C513694"
 			(at 492.76 129.54 0)
 			(hide yes)
@@
 			)
 		)
-		(property "MPN" "RL0402FR-070R82L"
+		(property "MPN" "RL0805FR-070R82L"
 			(at 492.76 129.54 0)
 			(hide yes)
@@
 			)
 		)
-		(property "Footprint" "Resistor_SMD:R_0402_1005Metric"
+		(property "Footprint" "Resistor_SMD:R_0805_2012Metric"
 			(at 543.56 129.54 0)
 			(hide yes)
@@
 			)
 		)
-		(property "LCSC" "C728435"
+		(property "LCSC" "C513694"
 			(at 543.56 129.54 0)
 			(hide yes)
@@
 			)
 		)
-		(property "MPN" "RL0402FR-070R82L"
+		(property "MPN" "RL0805FR-070R82L"
 			(at 543.56 129.54 0)
 			(hide yes)
@@
 			)
 		)
-		(property "Footprint" "Resistor_SMD:R_0402_1005Metric"
+		(property "Footprint" "Resistor_SMD:R_0805_2012Metric"
 			(at 116.84 175.26 0)
 			(hide yes)
@@
 			)
 		)
-		(property "LCSC" "C728435"
+		(property "LCSC" "C513694"
 			(at 116.84 175.26 0)
 			(hide yes)
@@
 			)
 		)
-		(property "MPN" "RL0402FR-070R82L"
+		(property "MPN" "RL0805FR-070R82L"
 			(at 116.84 175.26 0)
 			(hide yes)
@@
 			)
 		)
-		(property "Footprint" "Resistor_SMD:R_0402_1005Metric"
+		(property "Footprint" "Resistor_SMD:R_0805_2012Metric"
 			(at 167.64 175.26 0)
 			(hide yes)
@@
 			)
 		)
-		(property "LCSC" "C728435"
+		(property "LCSC" "C513694"
 			(at 167.64 175.26 0)
 			(hide yes)
@@
 			)
 		)
-		(property "MPN" "RL0402FR-070R82L"
+		(property "MPN" "RL0805FR-070R82L"
 			(at 167.64 175.26 0)
 			(hide yes)
@@
 			)
 		)
-		(property "Footprint" "Resistor_SMD:R_0402_1005Metric"
+		(property "Footprint" "Resistor_SMD:R_0805_2012Metric"
 			(at 492.76 175.26 0)
 			(hide yes)
@@
 			)
 		)
-		(property "LCSC" "C728435"
+		(property "LCSC" "C513694"
 			(at 492.76 175.26 0)
 			(hide yes)
@@
 			)
 		)
-		(property "MPN" "RL0402FR-070R82L"
+		(property "MPN" "RL0805FR-070R82L"
 			(at 492.76 175.26 0)
 			(hide yes)
@@
 			)
 		)
-		(property "Footprint" "Resistor_SMD:R_0402_1005Metric"
+		(property "Footprint" "Resistor_SMD:R_0805_2012Metric"
 			(at 543.56 175.26 0)
 			(hide yes)
@@
 			)
 		)
-		(property "LCSC" "C728435"
+		(property "LCSC" "C513694"
 			(at 543.56 175.26 0)
 			(hide yes)
@@
 			)
 		)
-		(property "MPN" "RL0402FR-070R82L"
+		(property "MPN" "RL0805FR-070R82L"
 			(at 543.56 175.26 0)
 			(hide yes)
@@
 			)
 		)
-		(property "Footprint" "Resistor_SMD:R_0402_1005Metric"
+		(property "Footprint" "Resistor_SMD:R_0805_2012Metric"
 			(at 116.84 220.98 0)
 			(hide yes)
@@
 			)
 		)
-		(property "LCSC" "C728435"
+		(property "LCSC" "C513694"
 			(at 116.84 220.98 0)
 			(hide yes)
@@
 			)
 		)
-		(property "MPN" "RL0402FR-070R82L"
+		(property "MPN" "RL0805FR-070R82L"
 			(at 116.84 220.98 0)
 			(hide yes)
@@
 			)
 		)
-		(property "Footprint" "Resistor_SMD:R_0402_1005Metric"
+		(property "Footprint" "Resistor_SMD:R_0805_2012Metric"
 			(at 167.64 220.98 0)
 			(hide yes)
@@
 			)
 		)
-		(property "LCSC" "C728435"
+		(property "LCSC" "C513694"
 			(at 167.64 220.98 0)
 			(hide yes)
@@
 			)
 		)
-		(property "MPN" "RL0402FR-070R82L"
+		(property "MPN" "RL0805FR-070R82L"
 			(at 167.64 220.98 0)
 			(hide yes)
@@
 			)
 		)
-		(property "Footprint" "Resistor_SMD:R_0402_1005Metric"
+		(property "Footprint" "Resistor_SMD:R_0805_2012Metric"
 			(at 492.76 220.98 0)
 			(hide yes)
@@
 			)
 		)
-		(property "LCSC" "C728435"
+		(property "LCSC" "C513694"
 			(at 492.76 220.98 0)
 			(hide yes)
@@
 			)
 		)
-		(property "MPN" "RL0402FR-070R82L"
+		(property "MPN" "RL0805FR-070R82L"
 			(at 492.76 220.98 0)
 			(hide yes)
@@
 			)
 		)
-		(property "Footprint" "Resistor_SMD:R_0402_1005Metric"
+		(property "Footprint" "Resistor_SMD:R_0805_2012Metric"
 			(at 543.56 220.98 0)
 			(hide yes)
@@
 			)
 		)
-		(property "LCSC" "C728435"
+		(property "LCSC" "C513694"
 			(at 543.56 220.98 0)
 			(hide yes)
@@
 			)
 		)
-		(property "MPN" "RL0402FR-070R82L"
+		(property "MPN" "RL0805FR-070R82L"
 			(at 543.56 220.98 0)
 			(hide yes)

Commit message: single_sh: 0603 sense resistors; refilled zones, fab output
Sense resistors move from 0805 to 0603 (Viking SR731JTTDR820F, C186570,
250 mW); holding a coil at the current-limit trip is now 28 % of rating.
Swapped in place on the routed board: ISEN pad kept, GND pad 0.275 mm
inboard (R5/R11 keep the GND pad instead). Zones refilled after the route
cleanup and trace edits. DRC: 0 unconnected, 0 parity, no copper
violations; 4 silkscreen warnings.

Schematics, BOMs, generators and README updated; JLCPCB Gerbers/BOM/CPL
regenerated and placement-checked.

Co-Authored-By: Claude Opus 5.5 <noreply@anthropic.com>
Parts:
- R1, R10, R11, R12, R13, R14, R15, R16, R17, R18, R19, R2, R20, R3, R4, R5, R6, R7, R8, R9: footprint Resistor_SMD:R_0805_2012Metric -> Resistor_SMD:R_0603_1608Metric; LCSC C513694 -> C186570; MPN RL0805FR-070R82L -> SR731JTTDR820F
Changed lines of the file:
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@@
 			)
 		)
-		(property "Footprint" "Resistor_SMD:R_0805_2012Metric"
+		(property "Footprint" "Resistor_SMD:R_0603_1608Metric"
 			(at 116.84 40.64 0)
 			(hide yes)
@@
 			)
 		)
-		(property "LCSC" "C513694"
+		(property "LCSC" "C186570"
 			(at 116.84 40.64 0)
 			(hide yes)
@@
 			)
 		)
-		(property "MPN" "RL0805FR-070R82L"
+		(property "MPN" "SR731JTTDR820F"
 			(at 116.84 40.64 0)
 			(hide yes)
@@
 			)
 		)
-		(property "Footprint" "Resistor_SMD:R_0805_2012Metric"
+		(property "Footprint" "Resistor_SMD:R_0603_1608Metric"
 			(at 167.64 40.64 0)
 			(hide yes)
@@
 			)
 		)
-		(property "LCSC" "C513694"
+		(property "LCSC" "C186570"
 			(at 167.64 40.64 0)
 			(hide yes)
@@
 			)
 		)
-		(property "MPN" "RL0805FR-070R82L"
+		(property "MPN" "SR731JTTDR820F"
 			(at 167.64 40.64 0)
 			(hide yes)
@@
 			)
 		)
-		(property "Footprint" "Resistor_SMD:R_0805_2012Metric"
+		(property "Footprint" "Resistor_SMD:R_0603_1608Metric"
 			(at 492.76 40.64 0)
 			(hide yes)
@@
 			)
 		)
-		(property "LCSC" "C513694"
+		(property "LCSC" "C186570"
 			(at 492.76 40.64 0)
 			(hide yes)
@@
 			)
 		)
-		(property "MPN" "RL0805FR-070R82L"
+		(property "MPN" "SR731JTTDR820F"
 			(at 492.76 40.64 0)
 			(hide yes)
@@
 			)
 		)
-		(property "Footprint" "Resistor_SMD:R_0805_2012Metric"
+		(property "Footprint" "Resistor_SMD:R_0603_1608Metric"
 			(at 543.56 40.64 0)
 			(hide yes)
@@
 			)
 		)
-		(property "LCSC" "C513694"
+		(property "LCSC" "C186570"
 			(at 543.56 40.64 0)
 			(hide yes)
@@
 			)
 		)
-		(property "MPN" "RL0805FR-070R82L"
+		(property "MPN" "SR731JTTDR820F"
 			(at 543.56 40.64 0)
 			(hide yes)
@@
 			)
 		)
-		(property "Footprint" "Resistor_SMD:R_0805_2012Metric"
+		(property "Footprint" "Resistor_SMD:R_0603_1608Metric"
 			(at 116.84 86.36 0)
 			(hide yes)
@@
 			)
 		)
-		(property "LCSC" "C513694"
+		(property "LCSC" "C186570"
 			(at 116.84 86.36 0)
 			(hide yes)
@@
 			)
 		)
-		(property "MPN" "RL0805FR-070R82L"
+		(property "MPN" "SR731JTTDR820F"
 			(at 116.84 86.36 0)
 			(hide yes)
@@
 			)
 		)
-		(property "Footprint" "Resistor_SMD:R_0805_2012Metric"
+		(property "Footprint" "Resistor_SMD:R_0603_1608Metric"
 			(at 167.64 86.36 0)
 			(hide yes)
@@
 			)
 		)
-		(property "LCSC" "C513694"
+		(property "LCSC" "C186570"
 			(at 167.64 86.36 0)
 			(hide yes)
@@
 			)
 		)
-		(property "MPN" "RL0805FR-070R82L"
+		(property "MPN" "SR731JTTDR820F"
 			(at 167.64 86.36 0)
 			(hide yes)
@@
 			)
 		)
-		(property "Footprint" "Resistor_SMD:R_0805_2012Metric"
+		(property "Footprint" "Resistor_SMD:R_0603_1608Metric"
 			(at 492.76 86.36 0)
 			(hide yes)
@@
 			)
 		)
-		(property "LCSC" "C513694"
+		(property "LCSC" "C186570"
 			(at 492.76 86.36 0)
 			(hide yes)
@@
 			)
 		)
-		(property "MPN" "RL0805FR-070R82L"
+		(property "MPN" "SR731JTTDR820F"
 			(at 492.76 86.36 0)
 			(hide yes)
@@
 			)
 		)
-		(property "Footprint" "Resistor_SMD:R_0805_2012Metric"
+		(property "Footprint" "Resistor_SMD:R_0603_1608Metric"
 			(at 543.56 86.36 0)
 			(hide yes)
@@
 			)
 		)
-		(property "LCSC" "C513694"
+		(property "LCSC" "C186570"
 			(at 543.56 86.36 0)
 			(hide yes)
@@
 			)
 		)
-		(property "MPN" "RL0805FR-070R82L"
+		(property "MPN" "SR731JTTDR820F"
 			(at 543.56 86.36 0)
 			(hide yes)
@@
 			)
 		)
-		(property "Footprint" "Resistor_SMD:R_0805_2012Metric"
+		(property "Footprint" "Resistor_SMD:R_0603_1608Metric"
 			(at 116.84 129.54 0)
 			(hide yes)
@@
 			)
 		)
-		(property "LCSC" "C513694"
+		(property "LCSC" "C186570"
 			(at 116.84 129.54 0)
 			(hide yes)
@@
 			)
 		)
-		(property "MPN" "RL0805FR-070R82L"
+		(property "MPN" "SR731JTTDR820F"
 			(at 116.84 129.54 0)
 			(hide yes)
@@
 			)
 		)
-		(property "Footprint" "Resistor_SMD:R_0805_2012Metric"
+		(property "Footprint" "Resistor_SMD:R_0603_1608Metric"
 			(at 167.64 129.54 0)
 			(hide yes)
@@
 			)
 		)
-		(property "LCSC" "C513694"
+		(property "LCSC" "C186570"
 			(at 167.64 129.54 0)
 			(hide yes)
@@
 			)
 		)
-		(property "MPN" "RL0805FR-070R82L"
+		(property "MPN" "SR731JTTDR820F"
 			(at 167.64 129.54 0)
 			(hide yes)
@@
 			)
 		)
-		(property "Footprint" "Resistor_SMD:R_0805_2012Metric"
+		(property "Footprint" "Resistor_SMD:R_0603_1608Metric"
 			(at 492.76 129.54 0)
 			(hide yes)
@@
 			)
 		)
-		(property "LCSC" "C513694"
+		(property "LCSC" "C186570"
 			(at 492.76 129.54 0)
 			(hide yes)
@@
 			)
 		)
-		(property "MPN" "RL0805FR-070R82L"
+		(property "MPN" "SR731JTTDR820F"
 			(at 492.76 129.54 0)
 			(hide yes)
@@
 			)
 		)
-		(property "Footprint" "Resistor_SMD:R_0805_2012Metric"
+		(property "Footprint" "Resistor_SMD:R_0603_1608Metric"
 			(at 543.56 129.54 0)
 			(hide yes)
@@
 			)
 		)
-		(property "LCSC" "C513694"
+		(property "LCSC" "C186570"
 			(at 543.56 129.54 0)
 			(hide yes)
@@
 			)
 		)
-		(property "MPN" "RL0805FR-070R82L"
+		(property "MPN" "SR731JTTDR820F"
 			(at 543.56 129.54 0)
 			(hide yes)
@@
 			)
 		)
-		(property "Footprint" "Resistor_SMD:R_0805_2012Metric"
+		(property "Footprint" "Resistor_SMD:R_0603_1608Metric"
 			(at 116.84 175.26 0)
 			(hide yes)
@@
 			)
 		)
-		(property "LCSC" "C513694"
+		(property "LCSC" "C186570"
 			(at 116.84 175.26 0)
 			(hide yes)
@@
 			)
 		)
-		(property "MPN" "RL0805FR-070R82L"
+		(property "MPN" "SR731JTTDR820F"
 			(at 116.84 175.26 0)
 			(hide yes)
@@
 			)
 		)
-		(property "Footprint" "Resistor_SMD:R_0805_2012Metric"
+		(property "Footprint" "Resistor_SMD:R_0603_1608Metric"
 			(at 167.64 175.26 0)
 			(hide yes)
@@
 			)
 		)
-		(property "LCSC" "C513694"
+		(property "LCSC" "C186570"
 			(at 167.64 175.26 0)
 			(hide yes)
@@
 			)
 		)
-		(property "MPN" "RL0805FR-070R82L"
+		(property "MPN" "SR731JTTDR820F"
 			(at 167.64 175.26 0)
 			(hide yes)
@@
 			)
 		)
-		(property "Footprint" "Resistor_SMD:R_0805_2012Metric"
+		(property "Footprint" "Resistor_SMD:R_0603_1608Metric"
 			(at 492.76 175.26 0)
 			(hide yes)
@@
 			)
 		)
-		(property "LCSC" "C513694"
+		(property "LCSC" "C186570"
 			(at 492.76 175.26 0)
 			(hide yes)
@@
 			)
 		)
-		(property "MPN" "RL0805FR-070R82L"
+		(property "MPN" "SR731JTTDR820F"
 			(at 492.76 175.26 0)
 			(hide yes)
@@
 			)
 		)
-		(property "Footprint" "Resistor_SMD:R_0805_2012Metric"
+		(property "Footprint" "Resistor_SMD:R_0603_1608Metric"
 			(at 543.56 175.26 0)
 			(hide yes)
@@
 			)
 		)
-		(property "LCSC" "C513694"
+		(property "LCSC" "C186570"
 			(at 543.56 175.26 0)
 			(hide yes)
@@
 			)
 		)
-		(property "MPN" "RL0805FR-070R82L"
+		(property "MPN" "SR731JTTDR820F"
 			(at 543.56 175.26 0)
 			(hide yes)
@@
 			)
 		)
-		(property "Footprint" "Resistor_SMD:R_0805_2012Metric"
+		(property "Footprint" "Resistor_SMD:R_0603_1608Metric"
 			(at 116.84 220.98 0)
 			(hide yes)
@@
 			)
 		)
-		(property "LCSC" "C513694"
+		(property "LCSC" "C186570"
 			(at 116.84 220.98 0)
 			(hide yes)
@@
 			)
 		)
-		(property "MPN" "RL0805FR-070R82L"
+		(property "MPN" "SR731JTTDR820F"
 			(at 116.84 220.98 0)
 			(hide yes)
@@
 			)
 		)
-		(property "Footprint" "Resistor_SMD:R_0805_2012Metric"
+		(property "Footprint" "Resistor_SMD:R_0603_1608Metric"
 			(at 167.64 220.98 0)
 			(hide yes)
@@
 			)
 		)
-		(property "LCSC" "C513694"
+		(property "LCSC" "C186570"
 			(at 167.64 220.98 0)
 			(hide yes)
@@
 			)
 		)
-		(property "MPN" "RL0805FR-070R82L"
+		(property "MPN" "SR731JTTDR820F"
 			(at 167.64 220.98 0)
 			(hide yes)
@@
 			)
 		)
-		(property "Footprint" "Resistor_SMD:R_0805_2012Metric"
+		(property "Footprint" "Resistor_SMD:R_0603_1608Metric"
 			(at 492.76 220.98 0)
 			(hide yes)
@@
 			)
 		)
-		(property "LCSC" "C513694"
+		(property "LCSC" "C186570"
 			(at 492.76 220.98 0)
 			(hide yes)
@@
 			)
 		)
-		(property "MPN" "RL0805FR-070R82L"
+		(property "MPN" "SR731JTTDR820F"
 			(at 492.76 220.98 0)
 			(hide yes)
@@
 			)
 		)
-		(property "Footprint" "Resistor_SMD:R_0805_2012Metric"
+		(property "Footprint" "Resistor_SMD:R_0603_1608Metric"
 			(at 543.56 220.98 0)
 			(hide yes)
@@
 			)
 		)
-		(property "LCSC" "C513694"
+		(property "LCSC" "C186570"
 			(at 543.56 220.98 0)
 			(hide yes)
@@
 			)
 		)
-		(property "MPN" "RL0805FR-070R82L"
+		(property "MPN" "SR731JTTDR820F"
 			(at 543.56 220.98 0)
 			(hide yes)

Commit message: single_sh_proto: all-0603 basic-parts prototype board, as ordered
150 x 30 mm 4-layer board, fully routed (0.52/0.3 vias, 45-degree traces,
centred pad entries, no vias in pads), JLCDFM clean. Corrected nested
dual-motor connector pinout, bring-up test points, back-silk squid art.
L1 substituted (C411344); status LED D2 is the 5050 WS2812B (C2843785),
left off the Economic PCBA order for hand soldering.

Generator updates for the proto board (build.py, pcbgen.py, jlcfab.py,
single_sh_sch.py, add_testpoints.py, squid_silk.py) and regenerated
outputs for the other boards.

Ordered from JLCPCB 2026-10-11: 5 boards, Economic PCBA.

Co-Authored-By: Claude Opus 5.5 <noreply@anthropic.com>
Parts:
- R1, R10, R11, R12, R13, R14, R15, R16, R17, R18, R19, R2, R20, R3, R4, R5, R6, R7, R8, R9: value 0.82 -> 1; LCSC C186570 -> C22936; MPN SR731JTTDR820F -> 0603WAF100KT5E; Note chops at 0.2-0.29 A (VTRIP 160-240 mV); Kelvin return -> chops at 0.16-0.24 A (VTRIP 160-240 mV); Kelvin return
